Commit message: add camera to panda model

File: icub_model_pybullet/franka_panda/panda_model.urdf (robot description, URDF)
Before this commit: robot panda, 13 links, 12 joints
Links:
- added link camera_color_frame, mass 0.00001
- added link camera_color_optical_frame, mass 0.00001
- added link camera_depth_frame, mass 0.00001
- added link camera_depth_optical_frame, mass 0.00001
- added link camera_left_ir_frame, mass 0.00001
- added link camera_left_ir_optical_frame, mass 0.00001
- added link camera_link, mass 0.564; collision box size=0.02505 0.09 0.025; visual mesh filename=package://meshes/visual/d435.dae
- added link camera_right_ir_frame, mass 0.00001
- added link camera_right_ir_optical_frame, mass 0.00001
Joints:
- added joint camera_color_joint: type fixed, parent camera_depth_frame, child camera_color_frame, origin xyz=0 0.015 0 rpy=0 0 0
- added joint camera_color_optical_joint: type fixed, parent camera_color_frame, child camera_color_optical_frame, origin xyz=0 0 0 rpy=-1.57079632679 0 -1.57079632679
- added joint camera_depth_joint: type fixed, parent camera_link, child camera_depth_frame, origin xyz=0.0149 0.0175 0.0125 rpy=0 0 0
- added joint camera_depth_optical_joint: type fixed, parent camera_depth_frame, child camera_depth_optical_frame, origin xyz=0 0 0 rpy=-1.57079632679 0 -1.57079632679
- added joint camera_joint: type fixed, parent panda_hand, child camera_link, origin xyz=0.027 0.0 0.02 rpy=0.0 -1.57 3.14
- added joint camera_left_ir_joint: type fixed, parent camera_depth_frame, child camera_left_ir_frame, origin xyz=0 0.0 0 rpy=0 0 0
- added joint camera_left_ir_optical_joint: type fixed, parent camera_left_ir_frame, child camera_left_ir_optical_frame, origin xyz=0 0 0 rpy=-1.57079632679 0 -1.57079632679
- added joint camera_right_ir_joint: type fixed, parent camera_depth_frame, child camera_right_ir_frame, origin xyz=0 -0.05 0 rpy=0 0 0
- added joint camera_right_ir_optical_joint: type fixed, parent camera_right_ir_frame, child camera_right_ir_optical_frame, origin xyz=0 0 0 rpy=-1.57079632679 0 -1.57079632679
